File: Hardware/Qwiic_keypad.brd (EAGLE design)
At the start: 25.4 x 25.4 mm, 36 parts, among them J3 PTH, J6 AVR_SPI_PROG_3X2TESTPOINTS, U3 ATTINY84

Commit message: remove wire stub
Routing:
- net 2: track 11.0 -> 10.5 mm
Changed lines of the file:
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@@
 <contactref element="U3" pad="12"/>
 <contactref element="J8" pad="2"/>
-<wire x1="13.335" y1="9.9" x2="13.335" y2="9.398" width="0.1524" layer="1"/>
 <wire x1="13.335" y1="9.9" x2="13.335" y2="8.35000625" width="0.1524" layer="1"/>
 <wire x1="13.335" y1="8.35000625" x2="17.78" y2="3.90500625" width="0.1524" layer="1"/>
