File: Hardware/Production/Qwiic_keypad-Panel.brd (EAGLE design)
At the start: 25.4 x 25.4 mm, 36 parts, among them J3 PTH, J6 AVR_SPI_PROG_3X2TESTPOINTS, U3 ATTINY84

Commit message: v2 update
Parts:
- removed FRAME1: FRAME-LETTER, SparkFun-Aesthetics:CREATIVE_COMMONS
- added C1, C2, C3, C5, C6, C7, C8, C9: 0.1uF, SparkFun-Capacitors:0603
- added D2, D3, D4, D5, D6, D7, D8, D9: RED, SparkFun-LED:LED-0603
- added E$1, E$2: (no value), SparkFun-Aesthetics:FIDUCIAL-1X2
- added E$3: (no value), SparkFun-Retired:FIDUCIAL-1.5X3
- added H10, H11, H12, H13, H14, H15, H16, H17, H18, H3, H4, H5, H6, H7, H8, H9: STAND-OFF, SparkFun-Hardware:STAND-OFF
- added J10, J15, J17, J22, J24, J29, J31, J36, J38, J43, J45, J50, J52, J57, J59, J7: (no value), SparkFun-Connectors:1X04_1MM_RA
- added J11, J13, J18, J20, J25, J27, J32, J34, J39, J41, J46, J48, J53, J55, J60, J62: (no value), SparkFun-Connectors:1X01_NO_SILK
- added J12, J19, J26, J33, J40, J47, J54, J61: AVR_SPI_PROG_3X2TESTPOINTS, SparkFun-Connectors:2X3_TEST_POINTS
- added J14, J21, J28, J35, J42, J49, J56, J63: (no value), SparkFun-Connectors:1X07_NO_SILK
- added J16, J23, J30, J37, J44, J51, J58, J9: PTH, SparkX:1X04_NO_SILK
- added JP10, JP15, JP20, JP25, JP30, JP35, JP40, JP45: (no value), SparkFun-Jumpers:SMT-JUMPER_2_NO_SILK
- added JP11, JP12, JP13, JP14, JP16, JP17, JP18, JP19, JP21, JP22, JP23, JP24, JP26, JP27, JP28, JP29, JP31, JP32, JP33, JP34, JP36, JP37, JP38, JP39, JP41, JP42, JP43, JP44, JP5, JP7, JP8, JP9: FIDUCIALUFIDUCIAL, SparkFun:MICRO-FIDUCIAL
- added LOGO2, LOGO3, LOGO4, LOGO5, LOGO6, LOGO7, LOGO8, LOGO9: OSHW-LOGOMINI, SparkFun-Aesthetics:OSHW-LOGO-MINI
- added R10, R14, R18, R22, R26, R30, R34, R5: 1k, SparkFun-Resistors:0603
- added R11, R12, R15, R16, R19, R20, R23, R24, R27, R28, R31, R32, R35, R36, R7, R8: 2.2k, SparkFun-Resistors:0603
- added R13, R17, R21, R25, R29, R33, R4, R9: 4.7k, SparkFun-Resistors:0603
- added SJ1, SJ2, SJ3, SJ4, SJ6, SJ7, SJ8, SJ9: (no value), SparkFun-Jumpers:SMT-JUMPER_3_NO_SILK
- added U$100, U$16, U$28, U$40, U$52, U$64, U$76, U$88: (no value), Labels-0_04:GND
- added U$101, U$17, U$29, U$41, U$53, U$65, U$77, U$89: (no value), Labels-0_04:SDA
- added U$102, U$18, U$30, U$42, U$54, U$66, U$78, U$90: (no value), Labels-0_04:SCL
- added U$103, U$19, U$31, U$43, U$55, U$67, U$79, U$91: (no value), Labels-0_04:(PWR)
- added U$104, U$20, U$32, U$44, U$56, U$68, U$80, U$92: (no value), Labels-0_04:(I_SUPER2_C)
- added U$105, U$21, U$33, U$45, U$57, U$69, U$81, U$93: (no value), Labels-0_04:(ADR)
- added U$106, U$22, U$34, U$46, U$58, U$70, U$82, U$94: (no value), Labels-0_04:#RST>
- added U$107, U$23, U$35, U$47, U$59, U$71, U$83, U$95: (no value), buzzard_labels (10):QWIIC_KEYPAD0
- added U$108, U$24, U$36, U$48, U$60, U$72, U$84, U$96: (no value), buzzard_labels (12):#INT1
- added U$13, U$25, U$26, U$37, U$38, U$49, U$50, U$61, U$62, U$7, U$73, U$74, U$85, U$86, U$97, U$98: SPARKX-LOGO3, SparkX:SPARKX-SMALL
- added U$14, U$27, U$39, U$51, U$63, U$75, U$87, U$99: (no value), Labels-0_04:3.3V
- added U1, U2, U4, U5, U6, U7, U8, U9: ATTINY84, SparkFun-IC-Microcontroller:SO14
- SJ5: device SparkFun-Jumpers:SMT-JUMPER_3_2-NC_TRACE_SILK -> SparkFun-Jumpers:SMT-JUMPER_3_NO_SILK
Connections:
- new net !INT1: J11.1, U1.6
- new net !INT2: J18.1, U2.6
- new net !INT3: J25.1, U4.6
- new net !INT4: J32.1, U5.6
- new net !INT5: J39.1, U6.6
- new net !INT6: J46.1, U7.6
- new net !INT7: J53.1, U8.6
- new net !INT8: J60.1, U9.6
- new net !RST1: J12.5, J13.1, R4.1, U1.4
- new net !RST2: J19.5, J20.1, R9.1, U2.4
- new net !RST3: J26.5, J27.1, R13.1, U4.4
- new net !RST4: J33.5, J34.1, R17.1, U5.4
- new net !RST5: J40.5, J41.1, R21.1, U6.4
- new net !RST6: J47.5, J48.1, R25.1, U7.4
- new net !RST7: J54.5, J55.1, R29.1, U8.4
- new net !RST8: J61.5, J62.1, R33.1, U9.4
- new net 10: J14.1, U1.13
- new net 11: J14.7, U1.2
- new net 12: J14.5, U1.5
- new net 13: J21.4, U2.10
- new net 14: J21.3, U2.11
- new net 15: J21.2, U2.12
- new net 16: J21.1, U2.13
- new net 17: J21.7, U2.2
- new net 18: J21.5, U2.5
- new net 19: J28.4, U4.10
- new net 20: J28.3, U4.11
- new net 21: J28.2, U4.12
- new net 22: J28.1, U4.13
- new net 23: J28.7, U4.2
- new net 24: J28.5, U4.5
- new net 25: J35.4, U5.10
- new net 26: J35.3, U5.11
- new net 27: J35.2, U5.12
- new net 28: J35.1, U5.13
- new net 29: J35.7, U5.2
- new net 3.3V1: C1.1, J10.2, J12.2, J7.2, J9.2, R4.2, R5.2, SJ1.2, U1.1
- new net 3.3V2: C2.1, J15.2, J16.2, J17.2, J19.2, R10.2, R9.2, SJ2.2, U2.1
- new net 3.3V3: C3.1, J22.2, J23.2, J24.2, J26.2, R13.2, R14.2, SJ3.2, U4.1
- new net 3.3V4: C5.1, J29.2, J30.2, J31.2, J33.2, R17.2, R18.2, SJ4.2, U5.1
- new net 3.3V5: C6.1, J36.2, J37.2, J38.2, J40.2, R21.2, R22.2, SJ6.2, U6.1
- new net 3.3V6: C7.1, J43.2, J44.2, J45.2, J47.2, R25.2, R26.2, SJ7.2, U7.1
- new net 3.3V7: C8.1, J50.2, J51.2, J52.2, J54.2, R29.2, R30.2, SJ8.2, U8.1
- new net 3.3V8: C9.1, J57.2, J58.2, J59.2, J61.2, R33.2, R34.2, SJ9.2, U9.1
- new net 30: J35.5, U5.5
- new net 31: J42.4, U6.10
- new net 32: J42.3, U6.11
- new net 33: J42.2, U6.12
- new net 34: J42.1, U6.13
- new net 35: J42.7, U6.2
- new net 36: J42.5, U6.5
- new net 37: J49.4, U7.10
- new net 38: J49.3, U7.11
- new net 39: J49.2, U7.12
- new net 40: J49.1, U7.13
- new net 41: J49.7, U7.2
- new net 42: J49.5, U7.5
- new net 43: J56.4, U8.10
- new net 44: J56.3, U8.11
- new net 45: J56.2, U8.12
- new net 46: J56.1, U8.13
- new net 47: J56.7, U8.2
- new net 48: J56.5, U8.5
- new net 49: J63.4, U9.10
- new net 50: J63.3, U9.11
- new net 51: J63.2, U9.12
- new net 52: J63.1, U9.13
- new net 53: J63.7, U9.2
- new net 54: J63.5, U9.5
- new net 6: J14.4, U1.10
- new net 8: J14.3, U1.11
- new net 9: J14.2, U1.12
- new net ADD2: JP10.2, U1.3
- new net ADD3: JP15.2, U2.3
- new net ADD4: JP20.2, U4.3
- new net ADD5: JP25.2, U5.3
- new net ADD6: JP30.2, U6.3
- new net ADD7: JP35.2, U7.3
- new net ADD8: JP40.2, U8.3
- new net ADD9: JP45.2, U9.3
- new net GND1: C1.2, D2.C, J10.1, J12.6, J7.1, J9.1, JP10.1, U1.14
- new net GND2: C2.2, D3.C, J15.1, J16.1, J17.1, J19.6, JP15.1, U2.14
- new net GND3: C3.2, D4.C, J22.1, J23.1, J24.1, J26.6, JP20.1, U4.14
- new net GND4: C5.2, D5.C, J29.1, J30.1, J31.1, J33.6, JP25.1, U5.14
- new net GND5: C6.2, D6.C, J36.1, J37.1, J38.1, J40.6, JP30.1, U6.14
- new net GND6: C7.2, D7.C, J43.1, J44.1, J45.1, J47.6, JP35.1, U7.14
- new net GND7: C8.2, D8.C, J50.1, J51.1, J52.1, J54.6, JP40.1, U8.14
- new net GND8: C9.2, D9.C, J57.1, J58.1, J59.1, J61.6, JP45.1, U9.14
- new net MISO/1: J12.1, J14.6, U1.8
- new net MISO/2: J19.1, J21.6, U2.8
- new net MISO/3: J26.1, J28.6, U4.8
- new net MISO/4: J33.1, J35.6, U5.8
- new net MISO/5: J40.1, J42.6, U6.8
- new net MISO/7: J47.1, J49.6, U7.8
- new net MISO/8: J54.1, J56.6, U8.8
- new net MISO/9: J61.1, J63.6, U9.8
- new net N$10: D4.A, R14.1
- new net N$11: R15.2, SJ3.3
- new net N$12: R16.2, SJ3.1
- new net N$13: D5.A, R18.1
- new net N$14: R19.2, SJ4.3
- new net N$15: R20.2, SJ4.1
- new net N$16: D6.A, R22.1
- new net N$17: R23.2, SJ6.3
- new net N$18: R24.2, SJ6.1
- new net N$19: D7.A, R26.1
- new net N$20: R27.2, SJ7.3
- new net N$21: R28.2, SJ7.1
- new net N$22: D8.A, R30.1
- new net N$23: R31.2, SJ8.3
- new net N$24: R32.2, SJ8.1
- new net N$25: D9.A, R34.1
- new net N$26: R35.2, SJ9.3
- new net N$27: R36.2, SJ9.1
- new net N$4: D2.A, R5.1
- new net N$5: R7.2, SJ1.3
- new net N$6: R8.2, SJ1.1
- new net N$7: D3.A, R10.1
- new net N$8: R11.2, SJ2.3
- new net N$9: R12.2, SJ2.1
- new net SCL1: J10.4, J12.3, J7.4, J9.4, R8.1, U1.9
- new net SCL2: J15.4, J16.4, J17.4, J19.3, R12.1, U2.9
- new net SCL3: J22.4, J23.4, J24.4, J26.3, R16.1, U4.9
- new net SCL4: J29.4, J30.4, J31.4, J33.3, R20.1, U5.9
- new net SCL5: J36.4, J37.4, J38.4, J40.3, R24.1, U6.9
- new net SCL6: J43.4, J44.4, J45.4, J47.3, R28.1, U7.9
- new net SCL7: J50.4, J51.4, J52.4, J54.3, R32.1, U8.9
- new net SCL8: J57.4, J58.4, J59.4, J61.3, R36.1, U9.9
- new net SDA1: J10.3, J12.4, J7.3, J9.3, R7.1, U1.7
- new net SDA2: J15.3, J16.3, J17.3, J19.4, R11.1, U2.7
- new net SDA3: J22.3, J23.3, J24.3, J26.4, R15.1, U4.7
- new net SDA4: J29.3, J30.3, J31.3, J33.4, R19.1, U5.7
- new net SDA5: J36.3, J37.3, J38.3, J40.4, R23.1, U6.7
- new net SDA6: J43.3, J44.3, J45.3, J47.4, R27.1, U7.7
- new net SDA7: J50.3, J51.3, J52.3, J54.4, R31.1, U8.7
- new net SDA8: J57.3, J58.3, J59.3, J61.4, R35.1, U9.7
Routing:
- net SDA8: track 0.00 -> 57.2 mm, vias 0 -> 2
- net SDA2: track 0.00 -> 57.2 mm, vias 0 -> 2
- net SDA7: track 0.00 -> 57.2 mm, vias 0 -> 2
- net SDA6: track 0.00 -> 57.2 mm, vias 0 -> 2
- net SDA5: track 0.00 -> 57.2 mm, vias 0 -> 2
- net SDA1: track 0.00 -> 57.2 mm, vias 0 -> 2
- net SDA4: track 0.00 -> 57.2 mm, vias 0 -> 2
- net SDA3: track 0.00 -> 57.2 mm, vias 0 -> 2
- net 3.3V8: track 0.00 -> 55.6 mm, vias 0 -> 4
- net 3.3V7: track 0.00 -> 55.6 mm, vias 0 -> 4
- net 3.3V2: track 0.00 -> 55.6 mm, vias 0 -> 4
- net 3.3V6: track 0.00 -> 55.6 mm, vias 0 -> 4
- net 3.3V5: track 0.00 -> 55.6 mm, vias 0 -> 4
- net 3.3V1: track 0.00 -> 55.6 mm, vias 0 -> 4
- net 3.3V4: track 0.00 -> 55.6 mm, vias 0 -> 4
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- added copper zone on layer 1, net GND1
- added copper zone on layer 16, net GND1
- added copper zone on layer 1, net GND2
- added copper zone on layer 16, net GND2
- added copper zone on layer 1, net GND3
- added copper zone on layer 16, net GND3
- added copper zone on layer 1, net GND4
- added copper zone on layer 16, net GND4
- added copper zone on layer 1, net GND5
- added copper zone on layer 16, net GND5
- added copper zone on layer 1, net GND6
- added copper zone on layer 16, net GND6
- added copper zone on layer 1, net GND7
- added copper zone on layer 16, net GND7
- added copper zone on layer 1, net GND8
- added copper zone on layer 16, net GND8
Other:
- board size 25.4 x 25.4 mm -> 97.3 x 97.3 mm
- board text added: "v-score"
- board text removed: "Kevin Kuwata"

Commit message: update panel and cam files
update to normally closed i2c jumper
Parts:
- SJ1, SJ2, SJ3, SJ4, SJ5, SJ6, SJ7, SJ8, SJ9: device SparkFun-Jumpers:SMT-JUMPER_3_NO_SILK -> SparkFun-Jumpers:SMT-JUMPER_3_2-NC_TRACE_SILK
Routing:
- net 51: track 11.0 -> 10.5 mm
- net 45: track 11.0 -> 10.5 mm
- net 39: track 11.0 -> 10.5 mm
- net 33: track 11.0 -> 10.5 mm
- net 27: track 11.0 -> 10.5 mm
- net 21: track 11.0 -> 10.5 mm
- net 15: track 11.0 -> 10.5 mm
- net 9: track 11.0 -> 10.5 mm
- net 2: track 11.0 -> 10.5 mm
